Commit message: Wheels Bigger

File: description/properties.xacro (robot description, xacro)
@@ -4,7 +4,9 @@
     <xacro:property name="chassis_thick"    value="0.05"/>     <!-- chassis height -->
     <xacro:property name="wheel_radius"     value="0.035"/>    <!-- ~70 mm dia. 0.035 -->
-    <xacro:property name="wheel_width"      value="0.01"/>
-    <xacro:property name="wheel_y_offset"   value="0.16"/>     <!-- offset from center -->
+    <xacro:property name="wheel_width"      value="0.05"/>      <!-- 0.01 -->
+    <xacro:property name="wheel_y_offset"   value="0.14"/>     <!-- offset from center  0.16-->
     <xacro:property name="caster_radius"    value="0.02"/> <!--0.02 -->
+    <!-- <xacro:property name="max_wheel_movement_down" value="${(chassis_radius*chassis_radius) - (wheel_y_offset*wheel_y_offset)}"/> -->
+    <xacro:property name="max_wheel_movement_down" value="0.03"/>
     <xacro:property name="caster_x_offset"  value="0.15"/>
     <xacro:property name="wheel_z" value="${(wheel_radius - (chassis_thick/2))-0.01}"/>

File: description/robot_core.xacro (robot description, xacro)
@@ -59,5 +59,5 @@
     <child link="left_wheel"/>
     <!-- lift wheel by its radius, rotate 90° (this is in radians, and 1.57 radians ~ 90deg or pi/2) around Y to align cylinder axis -->
-    <origin xyz="0 ${wheel_y_offset} ${wheel_z}" rpy="1.5708 0 0"/>
+    <origin xyz="${-max_wheel_movement_down} ${wheel_y_offset} ${wheel_z}" rpy="1.5708 0 0"/>
     <axis   xyz="0 0 1"/>
   </joint>
@@ -89,5 +89,5 @@
     <parent link="base_link"/>
     <child link="right_wheel"/>
-    <origin xyz="0 -${wheel_y_offset} ${wheel_z}" rpy="1.5708 0 0"/>
+    <origin xyz="${-max_wheel_movement_down} -${wheel_y_offset} ${wheel_z}" rpy="1.5708 0 0"/>
     <axis   xyz="0 0 1"/>
   </joint>
@@ -143,5 +143,5 @@
     <mu2 value="0.001"/>
   </gazebo>
-  <!-- <joint name="caster_wheel_joint_invisible" type="fixed">
+  <joint name="caster_wheel_joint_invisible" type="fixed">
     <parent link="base_link"/>
     <child link="caster_wheel_invisible"/>
@@ -171,5 +171,5 @@
     <mu2 value="0.001"/>
   </gazebo>
-  <joint name="caster_wheel_joint_invisible_l" type="fixed">
+  <!-- <joint name="caster_wheel_joint_invisible_l" type="fixed">
     <parent link="base_link"/>
     <child link="caster_wheel_invisible_l"/>
@@ -198,6 +198,6 @@
     <mu1 value="0.001"/>
     <mu2 value="0.001"/>
-  </gazebo>
-  <joint name="caster_wheel_joint_invisible_r" type="fixed">
+  </gazebo> -->
+  <!-- <joint name="caster_wheel_joint_invisible_r" type="fixed">
     <parent link="base_link"/>
     <child link="caster_wheel_invisible_r"/>

Commit message: Tried to fix movement again

File: description/properties.xacro (robot description, xacro)
@@ -4,9 +4,9 @@
     <xacro:property name="chassis_thick"    value="0.05"/>     <!-- chassis height -->
     <xacro:property name="wheel_radius"     value="0.035"/>    <!-- ~70 mm dia. 0.035 -->
-    <xacro:property name="wheel_width"      value="0.05"/>      <!-- 0.01 -->
-    <xacro:property name="wheel_y_offset"   value="0.14"/>     <!-- offset from center  0.16-->
+    <xacro:property name="wheel_width"      value="0.065"/>      <!-- 0.01 -->
+    <xacro:property name="wheel_y_offset"   value="0.12"/>     <!-- offset from center  0.16-->
     <xacro:property name="caster_radius"    value="0.02"/> <!--0.02 -->
     <!-- <xacro:property name="max_wheel_movement_down" value="${(chassis_radius*chassis_radius) - (wheel_y_offset*wheel_y_offset)}"/> -->
-    <xacro:property name="max_wheel_movement_down" value="0.03"/>
+    <xacro:property name="max_wheel_movement_down" value="0"/>
     <xacro:property name="caster_x_offset"  value="0.15"/>
     <xacro:property name="wheel_z" value="${(wheel_radius - (chassis_thick/2))-0.01}"/>

Commit message: Added Lazer

File: description/properties.xacro (robot description, xacro)
@@ -11,3 +11,7 @@
     <xacro:property name="caster_x_offset"  value="0.15"/>
     <xacro:property name="wheel_z" value="${(wheel_radius - (chassis_thick/2))-0.01}"/>
+    <xacro:property name="cam_length"   value="0.0405"/>
+    <xacro:property name="cam_width"   value="0.027"/>
+    <xacro:property name="cam_height"   value="0.0045"/>
+    <xacro:property name="ninety_deg"   value="1.5708"/>
 </robot>

File: description/robot.urdf.xacro (robot description, xacro)
@@ -3,3 +3,4 @@
     <xacro:include filename="robot_core.xacro"/>
     <xacro:include filename="gazebo_control.xacro"/>
+    <xacro:include filename="lidar.xacro"/>
 </robot>

File: description/robot_core.xacro (robot description, xacro)
@@ -22,4 +22,7 @@
       <color rgba="0 0 0 0"/>
     </material>
+    <material name="red">
+      <color rgba="1 0 0 1"/>
+    </material>
   <!--=== PROPERTIES ===-->
   <!-- All dimensions in meters -->

Commit message: Tried to balance robot

File: description/properties.xacro (robot description, xacro)
@@ -5,5 +5,5 @@
     <xacro:property name="wheel_radius"     value="0.035"/>    <!-- ~70 mm dia. 0.035 -->
     <xacro:property name="wheel_width"      value="0.065"/>      <!-- 0.01 -->
-    <xacro:property name="wheel_y_offset"   value="0.12"/>     <!-- offset from center  0.16-->
+    <xacro:property name="wheel_y_offset"   value="0.14"/>     <!-- offset from center  0.16-->
     <xacro:property name="caster_radius"    value="0.02"/> <!--0.02 -->
     <!-- <xacro:property name="max_wheel_movement_down" value="${(chassis_radius*chassis_radius) - (wheel_y_offset*wheel_y_offset)}"/> -->

File: description/robot_core.xacro (robot description, xacro)
@@ -117,6 +117,66 @@
     <material>Gazebo/Blue</material>
   </gazebo>
+  <joint name="right_wheel_joint_front" type="fixed">
+    <parent link="base_link"/>
+    <child link="right_wheel_front"/>
+    <origin xyz="${wheel_y_offset} 0 ${wheel_z}" rpy="1.5708 0 0"/>
+    <axis   xyz="0 0 1"/>
+  </joint>
+  <link name="right_wheel_front">
+    <visual>
+      <geometry>
+        <cylinder radius="${wheel_radius}" length="${wheel_width}"/>
+      </geometry>
+      <material name="orange"/>
+    </visual>
+    <collision>
+      <origin xyz="${wheel_y_offset} 0 ${wheel_z}" rpy="1.5708 0 0"/>
+      <geometry>
+        <cylinder radius="${wheel_radius}" length="${wheel_width}"/>
+      </geometry>
+    </collision>
+    <xacro:inertial_cylinder mass="0.15"
+                             length="${wheel_width}"
+                             radius="${wheel_radius}">
+      <origin rpy="1.5708 0 0"/>
+    </xacro:inertial_cylinder>
+  </link>
+  <gazebo reference="right_wheel_front">
+    <material>Gazebo/TransparentOrange</material>
+    <mu1 value="0.001"/>
+    <mu2 value="0.001"/>
+  </gazebo>
+  <joint name="left_wheel_joint_front" type="fixed">
+    <parent link="base_link"/>
+    <child link="left_wheel_front"/>
+    <origin xyz="${-wheel_y_offset} 0 ${wheel_z}" rpy="1.5708 0 0"/>
+    <axis   xyz="0 0 1"/>
+  </joint>
+  <link name="left_wheel_front">
+    <visual>
+      <geometry>
+        <cylinder radius="${wheel_radius}" length="${wheel_width}"/>
+      </geometry>
+      <material name="orange"/>
+    </visual>
+    <collision>
+      <origin xyz="${-wheel_y_offset} 0 ${wheel_z}" rpy="1.5708 0 0"/>
+      <geometry>
+        <cylinder radius="${wheel_radius}" length="${wheel_width}"/>
+      </geometry>
+    </collision>
+    <xacro:inertial_cylinder mass="0.15"
+                             length="${wheel_width}"
+                             radius="${wheel_radius}">
+      <origin rpy="1.5708 0 0"/>
+    </xacro:inertial_cylinder>
+  </link>
+  <gazebo reference="left_wheel_front">
+    <material>Gazebo/TransparentOrange</material>
+    <mu1 value="0.001"/>
+    <mu2 value="0.001"/>
+  </gazebo>
   <!--=== CASTER WHEEL ===-->
-  <joint name="caster_wheel_joint" type="fixed">
+  <!-- <joint name="caster_wheel_joint" type="fixed">
     <parent link="base_link"/>
     <child link="caster_wheel"/>
@@ -145,6 +205,6 @@
     <mu1 value="0.001"/>
     <mu2 value="0.001"/>
-  </gazebo>
-  <joint name="caster_wheel_joint_invisible" type="fixed">
+  </gazebo> -->
+  <!-- <joint name="caster_wheel_joint_invisible" type="fixed">
     <parent link="base_link"/>
     <child link="caster_wheel_invisible"/>
@@ -173,5 +233,5 @@
     <mu1 value="0.001"/>
     <mu2 value="0.001"/>
-  </gazebo>
+  </gazebo> -->
   <!-- <joint name="caster_wheel_joint_invisible_l" type="fixed">
     <parent link="base_link"/>

Commit message: Real Robot Movement with Rviz2

File: description/properties.xacro (robot description, xacro)
@@ -3,6 +3,6 @@
     <xacro:property name="chassis_radius"   value="0.1778"/>   <!-- 7 in = 0.1778 m -->
     <xacro:property name="chassis_thick"    value="0.05"/>     <!-- chassis height -->
-    <xacro:property name="wheel_radius"     value="0.035"/>    <!-- ~70 mm dia. 0.035 -->
-    <xacro:property name="wheel_width"      value="0.065"/>      <!-- 0.01 -->
+    <xacro:property name="wheel_radius"     value="0.0301625"/>    <!-- ~70 mm dia. 0.035 meters -->
+    <xacro:property name="wheel_width"      value="0.01905"/>      <!-- 0.01 -->
     <xacro:property name="wheel_y_offset"   value="0.14"/>     <!-- offset from center  0.16-->
     <xacro:property name="caster_radius"    value="0.02"/> <!--0.02 -->

File: description/ros2_control.xacro (robot description, xacro)
@@ -4,28 +4,24 @@
         <ros2_control name="RealRobot" type="system">
             <hardware>
-                <plugin>diffdrive_esp/DiffDriveEsp</plugin>
-                <param name="left_wheel_name">left_wheel_joint</param>
-                <param name="right_wheel_name">right_wheel_joint</param>
-                <param name="loop_rate">30</param>
-                <param name="device">/dev/ttyUSB0</param>
-                <param name="baud_rate">115200</param>
-                <!-- Serial_timeout 1000 = 1ms -->
-                <param name="timeout">1000</param>
-                <!-- Wheel revolutions, you'll need to modify this to match it -->
-                <param name="enc_counts_per_rev">3450</param>
+                <!-- Pulling our data from the robot itself with commands like /encoders -->
+                <plugin>fake_components/GenericSystem</plugin>
+                <!-- publish_rate controls how often the “fake” system polls for/advertises state -->
+                <param name="publish_rate">30</param>
+                <!-- tell it which joints exist -->
+                <param name="joint_names">['left_wheel_joint', 'right_wheel_joint']</param>
             </hardware>
             <joint name="left_wheel_joint">
-                <command_interface name="velocity">
-                    <param name="min">-10</param>
+                <command_interface name="velocity"/>
+                    <!-- <param name="min">-10</param>
                     <param name="max">10</param>
-                </command_interface>
+                </command_interface> -->
                 <state_interface name="velocity"/>
                 <state_interface name="position"/>
             </joint>
             <joint name="right_wheel_joint">
-                <command_interface name="velocity">
-                    <param name="min">-10</param>
-                    <param name="max">10</param>
-                </command_interface>
+                <command_interface name="velocity"/>
+                    <!-- <param name="min">-10</param>
+                    <param name="max">10</param> -->
+                <!-- </command_interface> -->
                 <state_interface name="velocity"/>
                 <state_interface name="position"/>
