Commit message: First Draft SLAM Setup

File: description/robot_core.xacro (robot description, xacro)
@@ -55,4 +55,11 @@
     <gravity>false</gravity>
   </gazebo>
+  <joint name="base_footprint_joint" type="fixed">
+        <parent link="base_link"/>
+        <child link="base_footprint"/>
+        <origin xyz="0 0 0" rpy="0 0 0"/>
+    </joint>
+  <link name="base_footprint">
+  </link>
   <!--=== LEFT WHEEL ===-->
   <!-- base_link then left_wheel_joint then left_wheel -->
